File: PCB-EAGLE/IndustrialUSBtoModbus.sch (EAGLE design)
At the start: 51 parts, among them IC10 ADUM1201ARZ, IC11 ADUM1201ARZ, IC2 MAX485CSA+, IC4 FT231XS-R

Commit message: feat: update USB RS485 hardware revision
Parts:
- removed R7: 120, SamacSys_Parts:ESR10EZPJ121
- added R4, R8: 5.1k, AKCP:ERJ-H3EF3300V
Connections:
- removed net N$16: R7.2, S1.S2A
- new net CC1: R4.2, USB.CC1
- new net CC2: R8.2, USB.CC2
- net B: no longer R7.1
- net GND: now also R4.1, R8.1
- net N$15: now also S1.S2A
Changed lines of the file:
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@@
 <?xml version="1.0" encoding="utf-8"?>
 <!DOCTYPE eagle SYSTEM "eagle.dtd">
-<eagle version="9.6.2">
+<eagle version="9.7.0">
 <drawing>
 <settings>
@@
 <setting verticaltext="up"/>
 </settings>
-<grid distance="0.1" unitdist="inch" unit="inch" style="lines" multiple="1" display="no" altdistance="0.01" altunitdist="inch" altunit="inch"/>
+<grid distance="0.01" unitdist="inch" unit="inch" style="lines" multiple="1" display="no" altdistance="0.01" altunitdist="inch" altunit="inch"/>
 <layers>
 <layer number="1" name="Top" color="4" fill="1" visible="no" active="no"/>
-<layer number="2" name="Route2" color="1" fill="3" visible="no" active="no"/>
-<layer number="3" name="Route3" color="4" fill="3" visible="no" active="no"/>
-<layer number="4" name="Route4" color="1" fill="4" visible="no" active="no"/>
-<layer number="5" name="Route5" color="4" fill="4" visible="no" active="no"/>
-<layer number="6" name="Route6" color="1" fill="8" visible="no" active="no"/>
-<layer number="7" name="Route7" color="4" fill="8" visible="no" active="no"/>
-<layer number="8" name="Route8" color="1" fill="2" visible="no" active="no"/>
-<layer number="9" name="Route9" color="4" fill="2" visible="no" active="no"/>
-<layer number="10" name="Route10" color="1" fill="7" visible="no" active="no"/>
-<layer number="11" name="Route11" color="4" fill="7" visible="no" active="no"/>
-<layer number="12" name="Route12" color="1" fill="5" visible="no" active="no"/>
-<layer number="13" name="Route13" color="4" fill="5" visible="no" active="no"/>
-<layer number="14" name="Route14" color="1" fill="6" visible="no" active="no"/>
-<layer number="15" name="Route15" color="4" fill="6" visible="no" active="no"/>
+<layer number="2" name="Route2" color="16" fill="3" visible="no" active="no"/>
+<layer number="3" name="Route3" color="17" fill="3" visible="no" active="no"/>
+<layer number="4" name="Route4" color="18" fill="4" visible="no" active="no"/>
+<layer number="5" name="Route5" color="19" fill="4" visible="no" active="no"/>
+<layer number="6" name="Route6" color="25" fill="8" visible="no" active="no"/>
+<layer number="7" name="Route7" color="26" fill="8" visible="no" active="no"/>
+<layer number="8" name="Route8" color="27" fill="2" visible="no" active="no"/>
+<layer number="9" name="Route9" color="28" fill="2" visible="no" active="no"/>
+<layer number="10" name="Route10" color="29" fill="7" visible="no" active="no"/>
+<layer number="11" name="Route11" color="30" fill="7" visible="no" active="no"/>
+<layer number="12" name="Route12" color="20" fill="5" visible="no" active="no"/>
+<layer number="13" name="Route13" color="21" fill="5" visible="no" active="no"/>
+<layer number="14" name="Route14" color="22" fill="6" visible="no" active="no"/>
+<layer number="15" name="Route15" color="23" fill="6" visible="no" active="no"/>
 <layer number="16" name="Bottom" color="1" fill="1" visible="no" active="no"/>
 <layer number="17" name="Pads" color="2" fill="1" visible="no" active="no"/>
 <layer number="18" name="Vias" color="2" fill="1" visible="no" active="no"/>
 <layer number="19" name="Unrouted" color="6" fill="1" visible="no" active="no"/>
-<layer number="20" name="Dimension" color="15" fill="1" visible="no" active="no"/>
+<layer number="20" name="Dimension" color="24" fill="1" visible="no" active="no"/>
 <layer number="21" name="tPlace" color="7" fill="1" visible="no" active="no"/>
 <layer number="22" name="bPlace" color="7" fill="1" visible="no" active="no"/>
@@
 <attribute name="SPICEPREFIX" value="R"/>
 </part>
-<part name="R7" library="SamacSys_Parts" library_urn="urn:adsk.eagle:library:22641528" deviceset="ESR10EZPJ121" device="" package3d_urn="urn:adsk.eagle:package:22798771/3" value="120">
-<attribute name="SPICEPREFIX" value="R"/>
-</part>
 <part name="S1" library="SamacSys_Parts" library_urn="urn:adsk.eagle:library:22550427" deviceset="210-2MS" device="" package3d_urn="urn:adsk.eagle:package:22550533/2">
 <attribute name="SPICEPREFIX" value="S"/>
@@
 <part name="+3V5" library="supply1" library_urn="urn:adsk.eagle:library:371" deviceset="+3V3" device=""/>
 <part name="GND13" library="DecawaveLibrary" library_urn="urn:adsk.eagle:library:5224885" deviceset="GND" device=""/>
+<part name="R4" library="AKCP" library_urn="urn:adsk.eagle:library:37273378" deviceset="ERJ-H3EF3300V" device="" package3d_urn="urn:adsk.eagle:package:37185905/2" value="5.1k"/>
+<part name="GND14" library="DecawaveLibrary" library_urn="urn:adsk.eagle:library:5224885" deviceset="GND" device=""/>
+<part name="R8" library="AKCP" library_urn="urn:adsk.eagle:library:37273378" deviceset="ERJ-H3EF3300V" device="" package3d_urn="urn:adsk.eagle:package:37185905/2" value="5.1k"/>
 </parts>
 <sheets>
@@
 <attribute name="VALUE" x="147.5994" y="155.4988" size="1.016" layer="96" align="center-left"/>
 </instance>
-<instance part="R7" gate="G$1" x="139.2174" y="152.9588" smashed="yes">
-<attribute name="NAME" x="144.2974" y="153.2128" size="1.016" layer="95" align="center-left"/>
-<attribute name="VALUE" x="147.5994" y="152.9588" size="1.016" layer="96" align="center-left"/>
-</instance>
 <instance part="S1" gate="G$1" x="158.2674" y="155.4988" smashed="yes">
 <attribute name="NAME" x="177.3174" y="159.3088" size="1.016" layer="95" align="center-left"/>
@@
 <instance part="GND13" gate="1" x="82.4738" y="63.0682" smashed="yes" rot="R270">
 <attribute name="VALUE" x="84.4296" y="64.77" size="1.016" layer="96" align="top-center"/>
+</instance>
+<instance part="R4" gate="G$1" x="15.6718" y="35.179" smashed="yes" rot="R270">
+<attribute name="NAME" x="15.6718" y="29.337" size="1.016" layer="95" rot="R270" align="center-left"/>
+<attribute name="VALUE" x="15.6718" y="25.273" size="1.016" layer="96" rot="R270" align="center-left"/>
+</instance>
+<instance part="GND14" gate="1" x="17.3482" y="38.9128" smashed="yes" rot="R180">
+<attribute name="VALUE" x="17.3482" y="39.1668" size="1.016" layer="96" rot="R180" align="top-center"/>
+</instance>
+<instance part="R8" gate="G$1" x="18.7198" y="35.179" smashed="yes" rot="R270">
+<attribute name="NAME" x="18.7198" y="29.337" size="1.016" layer="95" rot="R270" align="center-left"/>
+<attribute name="VALUE" x="18.7198" y="25.273" size="1.016" layer="96" rot="R270" align="center-left"/>
 </instance>
 </instances>
@@
 <wire x1="85.0138" y1="63.0682" x2="85.6742" y2="63.0682" width="0.1524" layer="91"/>
 <junction x="85.0138" y="63.0682"/>
+</segment>
+<segment>
+<pinref part="R4" gate="G$1" pin="1"/>
+<wire x1="15.6718" y1="35.179" x2="15.6718" y2="36.3728" width="0.1524" layer="91"/>
+<wire x1="15.6718" y1="36.3728" x2="17.3482" y2="36.3728" width="0.1524" layer="91"/>
+<pinref part="GND14" gate="1" pin="GND"/>
+<pinref part="R8" gate="G$1" pin="1"/>
+<wire x1="18.7198" y1="35.179" x2="18.7198" y2="36.3728" width="0.1524" layer="91"/>
+<wire x1="18.7198" y1="36.3728" x2="17.3482" y2="36.3728" width="0.1524" layer="91"/>
+<junction x="17.3482" y="36.3728"/>
 </segment>
 </net>
@@
 <segment>
 <pinref part="R6" gate="G$1" pin="1"/>
-<wire x1="139.2174" y1="155.4988" x2="137.9474" y2="155.4988" width="0.1524" layer="91"/>
-<wire x1="137.9474" y1="155.4988" x2="137.9474" y2="154.2288" width="0.1524" layer="91"/>
-<pinref part="R7" gate="G$1" pin="1"/>
-<wire x1="137.9474" y1="154.2288" x2="137.9474" y2="152.9588" width="0.1524" layer="91"/>
-<wire x1="137.9474" y1="152.9588" x2="139.2174" y2="152.9588" width="0.1524" layer="91"/>
-<wire x1="137.9474" y1="154.2288" x2="137.1854" y2="154.2288" width="0.1524" layer="91"/>
-<junction x="137.9474" y="154.2288"/>
-<label x="137.1854" y="154.2288" size="1.016" layer="95" rot="R180" xref="yes"/>
+<wire x1="139.2174" y1="155.4988" x2="137.1854" y2="155.4988" width="0.1524" layer="91"/>
+<label x="137.1854" y="155.4988" size="1.016" layer="95" rot="R180" xref="yes"/>
 </segment>
 <segment>
@@
 <wire x1="156.9974" y1="155.4988" x2="158.2674" y2="155.4988" width="0.1524" layer="91"/>
 <pinref part="S1" gate="G$1" pin="S1A"/>
-</segment>
-</net>
-<net name="N$16" class="0">
-<segment>
+<wire x1="158.2674" y1="155.4988" x2="158.2674" y2="152.9588" width="0.1524" layer="91"/>
+<junction x="158.2674" y="155.4988"/>
 <pinref part="S1" gate="G$1" pin="S2A"/>
-<pinref part="R7" gate="G$1" pin="2"/>
-<wire x1="158.2674" y1="152.9588" x2="156.9974" y2="152.9588" width="0.1524" layer="91"/>
 </segment>
 </net>
@@
 </segment>
 </net>
+<net name="CC1" class="0">
+<segment>
+<pinref part="USB" gate="G$1" pin="CC1"/>
+<wire x1="77.1398" y1="32.385" x2="75.184" y2="32.385" width="0.1524" layer="91"/>
+<wire x1="75.184" y1="32.385" x2="75.184" y2="32.512" width="0.1524" layer="91"/>
+<label x="75.184" y="32.512" size="1.016" layer="95" rot="R180" xref="yes"/>
+</segment>
+<segment>
+<pinref part="R4" gate="G$1" pin="2"/>
+<wire x1="15.6718" y1="17.399" x2="15.6718" y2="16.256" width="0.1524" layer="91"/>
+<wire x1="15.6718" y1="16.256" x2="15.748" y2="16.256" width="0.1524" layer="91"/>
+<label x="15.748" y="16.256" size="1.016" layer="95" rot="R270" xref="yes"/>
+</segment>
+</net>
+<net name="CC2" class="0">
+<segment>
+<pinref part="USB" gate="G$1" pin="CC2"/>
+<wire x1="112.6998" y1="24.765" x2="114.554" y2="24.765" width="0.1524" layer="91"/>
+<wire x1="114.554" y1="24.765" x2="114.554" y2="24.892" width="0.1524" layer="91"/>
+<label x="114.554" y="24.892" size="1.016" layer="95" rot="MR180" xref="yes"/>
+</segment>
+<segment>
+<pinref part="R8" gate="G$1" pin="2"/>
+<wire x1="18.7198" y1="17.399" x2="18.7198" y2="16.256" width="0.1524" layer="91"/>
+<wire x1="18.7198" y1="16.256" x2="18.796" y2="16.256" width="0.1524" layer="91"/>
+<label x="18.796" y="16.256" size="1.016" layer="95" rot="R270" xref="yes"/>
+</segment>
+</net>
